Commit message: Reach feature parity with the uFactory xArm module (0.2.0)
Implements every software item in PLAN.md, derived from a comparison
against viam:ufactory. Hardware-validation items remain open.

Motion-service compatibility
- Custom arm gRPC servicer (arm_service.py) adding MoveThroughJointPositions,
  MoveThroughJointPositionsStreamed, and Get3DModels, which the Python SDK
  0.80 servicer lacks; swapped into the SDK registry at module start.
- Interpolated setpoint streaming (trajectory.py) with per-joint velocity and
  acceleration limits, MoveOptions and extra-key overrides, single in-flight
  operation manager (ops.py), stop() that cancels within one tick.
- Out-of-limit targets are rejected (clip_targets restores clipping).
- move_to_position delegates to a configured motion service.

Geometry and 3D models
- Collision boxes (default) or decimated vendor STL meshes in the served
  URDF, shipped via meshes_by_urdf_filepath; get_geometries; GLB models.
- Assets built from Seeed's reBot-DevArm at a pinned commit
  (tools/build_assets.py, assets/ATTRIBUTION.md).
- Gripper URDF with one prismatic finger joint and collision boxes; its
  kinematic input is now finger travel in metres (breaking).

Safety and diagnostics
- Damiao status decoding, automatic clearing of transient faults, decoded
  errors on hard faults, temperature warn/limit, software torque-limit
  collision stop, CAN watchdog, serial reconnect with state restore,
  bad_joints, experimental manual mode with URDF-based gravity compensation.

Gripper
- arm dependency attribute (inherits the bus), runtime speed/force
  DoCommands, grab_with_force, get/set position commands.

Packaging
- pytest suite against an in-memory motorbridge fake (79 tests), ruff,
  GitHub Actions for tests and tagged-release publishing, Makefile,
  run.sh --check, CHANGELOG, README rewrite including the comparison.

Co-Authored-By: Claude Fable 5.1 <noreply@anthropic.com>

File: src/rebot_b601/rebot_b601_dm.urdf (robot description, URDF)
Before this commit: robot rebot_b601_dm, 8 links, 7 joints
Links:
- link base_link: mass None -> 0.8366
- link end_link: mass None -> 0.5
- link link1: mass None -> 0.1613
- link link2: mass None -> 1.3266
- link link3: mass None -> 0.8353
- link link4: mass None -> 0.52
- link link5: mass None -> 0.383
- link link6: mass None -> 0.3663
